File: 5x5 Display/5x5 Display.kicad_sch (KiCad schematic)
At the start: 52 parts, among them U3 DRV1

Commit message: R1
Parts:
- C2, C5: value 30μF ≥28V -> 22μF ≥28V; LCSC Part # (none) -> C6119966
- D6, D7, D8, D9: LCSC Part # (none) -> C134981
- L1: LCSC Part # (none) -> C2047296
- L2: LCSC Part # (none) -> C184350
Changed lines of the file:
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@@
 	)
 	(junction
-		(at 115.57 58.42)
-		(diameter 0)
-		(color 0 0 0 0)
-	)
-	(junction
 		(at 203.2 30.48)
 		(diameter 0)
@@
 	(wire
 		(pts
+			(xy 114.3 58.42) (xy 116.84 58.42)
+		)
+		(stroke
+			(width 0)
+			(type default)
+		)
+	)
+	(wire
+		(pts
 			(xy 118.11 82.55) (xy 110.49 82.55)
 		)
@@
 	(wire
 		(pts
-			(xy 114.3 58.42) (xy 115.57 58.42)
-		)
-		(stroke
-			(width 0)
-			(type default)
-		)
-	)
-	(wire
-		(pts
 			(xy 222.25 69.85) (xy 222.25 74.93)
 		)
@@
 	(wire
 		(pts
-			(xy 115.57 58.42) (xy 116.84 58.42)
-		)
-		(stroke
-			(width 0)
-			(type default)
-		)
-	)
-	(wire
-		(pts
 			(xy 189.23 90.17) (xy 189.23 87.63)
 		)
@@
 			)
 		)
-		(property "Value" "30μF ≥28V"
+		(property "Value" "22μF ≥28V"
 			(at 168.91 73.6662 0)
 			(effects
@@
 			)
 		)
-		(property "LCSC Part #" ""
+		(property "LCSC Part #" "C6119966"
 			(at 166.37 72.39 0)
 			(effects
@@
 			)
 		)
+		(property "LCSC Part #" "C134981"
+			(at 59.69 101.6 0)
+			(effects
+				(font
+					(size 1.27 1.27)
+				)
+				(hide yes)
+			)
+		)
 		(pin "2"
 		)
@@
 			)
 		)
+		(property "LCSC Part #" "C134981"
+			(at 59.69 90.17 0)
+			(effects
+				(font
+					(size 1.27 1.27)
+				)
+				(hide yes)
+			)
+		)
 		(pin "2"
 		)
@@
 			)
 		)
-		(property "Value" "30μF ≥28V"
+		(property "Value" "22μF ≥28V"
 			(at 168.91 29.2162 0)
 			(effects
@@
 			)
 		)
-		(property "LCSC Part #" ""
+		(property "LCSC Part #" "C6119966"
 			(at 166.37 27.94 0)
 			(effects
@@
 			)
 		)
+		(property "LCSC Part #" "C134981"
+			(at 34.29 101.6 0)
+			(effects
+				(font
+					(size 1.27 1.27)
+				)
+				(hide yes)
+			)
+		)
 		(pin "2"
 		)
@@
 	(symbol
 		(lib_id "power:GND")
-		(at 115.57 58.42 0)
+		(at 114.3 58.42 0)
 		(unit 1)
 		(exclude_from_sim no)
@@
 		(dnp no)
 		(property "Reference" "#PWR0161"
-			(at 115.57 64.77 0)
+			(at 114.3 64.77 0)
 			(effects
 				(font
@@
 		)
 		(property "Value" "GND"
-			(at 115.57 61.976 0)
+			(at 114.3 61.976 0)
 			(effects
 				(font
@@
 		)
 		(property "Footprint" ""
-			(at 115.57 58.42 0)
+			(at 114.3 58.42 0)
 			(effects
 				(font
@@
 		)
 		(property "Datasheet" ""
-			(at 115.57 58.42 0)
+			(at 114.3 58.42 0)
 			(effects
 				(font
@@
 		)
 		(property "Description" "Power symbol creates a global label with name \"GND\" , ground"
-			(at 115.57 58.42 0)
+			(at 114.3 58.42 0)
 			(effects
 				(font
@@
 			)
 		)
+		(property "LCSC Part #" "C184350"
+			(at 207.01 74.93 90)
+			(effects
+				(font
+					(size 1.27 1.27)
+				)
+				(hide yes)
+			)
+		)
 		(pin "1"
 		)
@@
 			)
 		)
+		(property "LCSC Part #" "C134981"
+			(at 34.29 90.17 0)
+			(effects
+				(font
+					(size 1.27 1.27)
+				)
+				(hide yes)
+			)
+		)
 		(pin "2"
 		)
@@
 			(effects
 				(font
+					(size 1.27 1.27)
+				)
+				(hide yes)
+			)
+		)
+		(property "LCSC Part #" "C2047296"
+			(at 207.01 30.48 90)
+			(effects
+				(font
