File: 5x5 Display/5x5 Display.kicad_pcb (KiCad board)
At the start: 4 copper layers, 129.5 x 129.5 mm, 102 parts, among them U3 DRV1

Commit message: R1
Routing:
- net CLK: track 673.9 -> 655.2 mm
- added copper zone on F.Cu, net (none)
Other:
- board text removed: "5X5 DISPLAY PROTOTYPE"

Commit message: R2 board routed
Parts:
- removed FUSE1: TPS1663x (VQFN), Package_DFN_QFN:VQFN-24-1EP_4x4mm_P0.5mm_EP2.5x2.5mm_ThermalVias
- removed NT1, NT2: NT, NetTie:NetTie-2_SMD_Pad0.5mm
- removed R10: 1kΩ, Resistor_SMD:R_0603_1608Metric
- removed R11, R12, R13, R14: 1.5kΩ, Resistor_SMD:R_0603_1608Metric
- removed REG3: L78M05ABDT, Package_TO_SOT_SMD:TO-252-2
- removed TP1: VBUS, TestPoint:TestPoint_Pad_D1.5mm
- removed TP12: GND, TestPoint:TestPoint_Pad_D1.5mm
- removed TP3: CLK_LOW, TestPoint:TestPoint_Pad_D1.5mm
- removed TP6: +3.3v, TestPoint:TestPoint_Pad_D1.5mm
- removed TP7: +5v, TestPoint:TestPoint_Pad_D1.5mm
- removed TP8: LED LDO, TestPoint:TestPoint_Pad_D1.5mm
- removed U3: DRV1, Package_SON:WSON-8-1EP_2x2mm_P0.5mm_EP0.9x1.6mm
- removed kibuzzard-69632EEE: G***, kibuzzard-69632EEE
- removed kibuzzard-69632F12: G***, kibuzzard-69632F12
- removed kibuzzard-69632F20: G***, kibuzzard-69632F20
- removed kibuzzard-69632F6C: G***, kibuzzard-69632F6C
- removed kibuzzard-69632F9B: G***, kibuzzard-69632F9B
- removed kibuzzard-69633F6A: G***, kibuzzard-69633F6A
- removed kibuzzard-6963405F: G***, kibuzzard-6963405F
- removed kibuzzard-696340B6: G***, kibuzzard-696340B6
- removed kibuzzard-69634119: G***, kibuzzard-69634119
- removed kibuzzard-6963413C: G***, kibuzzard-6963413C
- removed kibuzzard-696556F9: G***, kibuzzard-696556F9
- removed kibuzzard-69655720: G***, kibuzzard-69655720
- removed kibuzzard-6965572F: G***, kibuzzard-6965572F
- removed kibuzzard-6965573A: G***, kibuzzard-6965573A
- removed kibuzzard-69655742: G***, kibuzzard-69655742
- removed kibuzzard-6965596D: G***, kibuzzard-6965596D
- removed kibuzzard-69655B36: G***, kibuzzard-69655B36
- added C10: 10uF, Capacitor_SMD:C_1206_3216Metric, B.Cu at (113.7, 110.5)
- added DRV1: DRV8837C, Package_SON:WSON-8-1EP_2x2mm_P0.5mm_EP0.9x1.6mm, B.Cu at (84.9, 111.1)
- added Q1: PMOS, Package_DFN_QFN:PQFN-8-EP_6x5mm_P1.27mm_Generic, B.Cu at (165.7, 110.5)
- added kibuzzard-696F07FC: G***, kibuzzard-696F07FC, B.Cu at (161.3, 117.5)
- added kibuzzard-696F080D: G***, kibuzzard-696F080D, B.Cu at (135.9, 117.5)
- added kibuzzard-696F081C: G***, kibuzzard-696F081C, B.Cu at (110.5, 117.5)
- added kibuzzard-696F082C: G***, kibuzzard-696F082C, B.Cu at (87.0, 117.5)
- added kibuzzard-696F097A: G***, kibuzzard-696F097A, B.Cu at (182.6, 108.3)
- added kibuzzard-696F0995: G***, kibuzzard-696F0995, B.Cu at (182.0, 112.7)
- added kibuzzard-696F09B6: G***, kibuzzard-696F09B6, B.Cu at (181.4, 110.5)
- added kibuzzard-696F0B33: G***, kibuzzard-696F0B33, B.Cu at (184.8, 117.5)
- C1: value 47nF -> 10uF; footprint Capacitor_SMD:C_0603_1608Metric -> Capacitor_SMD:C_1206_3216Metric
- C2: value 30μF ≥28V -> 10uF
- C3: footprint Capacitor_SMD:C_0603_1608Metric -> Capacitor_SMD:C_0805_2012Metric
- C4: value 30μF ≥10V -> 100nF; footprint Capacitor_SMD:C_1206_3216Metric -> Capacitor_SMD:C_0805_2012Metric
- C5: value 30μF ≥28V -> 47uF
- C6: value 100nF -> 47uF; footprint Capacitor_SMD:C_0603_1608Metric -> Capacitor_SMD:C_1206_3216Metric
- C7: value 30μF ≥10V -> 47pF; footprint Capacitor_SMD:C_1206_3216Metric -> Capacitor_SMD:C_0603_1608Metric
- C8: value 100nF ≥10V -> 68pF
- C9: value 330nF ≥28V -> 10uF; footprint Capacitor_SMD:C_0805_2012Metric -> Capacitor_SMD:C_1206_3216Metric
- D1: value POWER -> ≥33V; footprint LED_SMD:LED_0805_2012Metric -> Diode_SMD:D_SMA
- D2: value FUSE FAULT -> ≥33V; footprint LED_SMD:LED_0805_2012Metric -> Diode_SMD:D_SMA
- D3: value 3.3V FAULT -> 12V Zener; footprint LED_SMD:LED_0805_2012Metric -> Diode_SMD:D_SOD-123
- D4: value 5V FAULT -> ≥33V; footprint LED_SMD:LED_0805_2012Metric -> Diode_SMD:D_SMA
- D5: value CLOCK -> ≥33V; footprint LED_SMD:LED_0805_2012Metric -> Diode_SMD:D_SMA
- D6: value ≥33V -> 3.3V; footprint Diode_SMD:D_SMA -> LED_SMD:LED_0805_2012Metric
- D7: value ≥33V -> 5V; footprint Diode_SMD:D_SMA -> LED_SMD:LED_0805_2012Metric
- D8: value ≥33V -> CLK; footprint Diode_SMD:D_SMA -> LED_SMD:LED_0805_2012Metric
- D9: value ≥33V -> Schottky; footprint Diode_SMD:D_SMA -> Diode_SMD:D_SOD-123
- L1: value 2.2μH -> 10uH; footprint Inductor_SMD:L_6.3x6.3_H3 -> Inductor_SMD:L_TechFuse_SL0630
- L2: value 3.3μH -> 6.8uH; footprint Inductor_SMD:L_6.3x6.3_H3 -> Inductor_SMD:L_TechFuse_SL0630
- POGO3: value Right - Socket -> Bottom - Socket
- POGO4: value Bottom - Socket -> Right - Socket
- R1: value 1.5MΩ -> 33kΩ; footprint Resistor_SMD:R_0603_1608Metric -> Resistor_SMD:R_0805_2012Metric
- R2: value 430kΩ -> 100kΩ; footprint Resistor_SMD:R_0603_1608Metric -> Resistor_SMD:R_0805_2012Metric
- R3: value 75kΩ -> 13kΩ; footprint Resistor_SMD:R_0603_1608Metric -> Resistor_SMD:R_0805_2012Metric
- R4: value 5.6kΩ -> 100kΩ; footprint Resistor_SMD:R_0603_1608Metric -> Resistor_SMD:R_0805_2012Metric
- R5: footprint Resistor_SMD:R_0603_1608Metric -> Resistor_SMD:R_0805_2012Metric
- R6: value 68kΩ -> 120Ω; footprint Resistor_SMD:R_0603_1608Metric -> Resistor_SMD:R_0805_2012Metric
- R7: value 15kΩ -> 300Ω; footprint Resistor_SMD:R_0603_1608Metric -> Resistor_SMD:R_0805_2012Metric
- R8: value 110kΩ -> 120Ω; footprint Resistor_SMD:R_0603_1608Metric -> Resistor_SMD:R_0805_2012Metric
- R9: value 15kΩ -> 10kΩ; footprint Resistor_SMD:R_0603_1608Metric -> Resistor_SMD:R_0805_2012Metric
- REG1: value TPS56637 3.3v -> TPS54302; footprint TPS56637:TPS56637 VQFN-HR (10) -> Package_TO_SOT_SMD:SOT-23-6
- REG2: value TPS56637 5V -> TPS54302; footprint TPS56637:TPS56637 VQFN-HR (10) -> Package_TO_SOT_SMD:SOT-23-6
- moved D8 110.8 mm to (185.1, 112.7), turned to 0 degrees
- moved D9 91.5 mm to (86.4, 106.9), turned to 90 degrees
- moved D4 88.7 mm to (134.6, 28.6)
- moved D1 69.9 mm to (76.8, 86.4), turned to 90 degrees
- moved R8 66.6 mm to (188.6, 112.7), turned to 180 degrees
- moved C4 59.4 mm to (106.0, 107.3), turned to 0 degrees
- moved D6 59.0 mm to (185.1, 110.5)
- moved D2 56.8 mm to (194.9, 86.4), turned to 90 degrees
- moved G*** 56.4 mm to (136.1, 56.1)
- moved kibuzzard-69659941 56.4 mm to (136.1, 66.7)
- moved R6 49.5 mm to (188.6, 110.5)
- moved R7 47.1 mm to (188.6, 108.3), turned to 180 degrees
- moved R4 47.0 mm to (102.2, 110.5), turned to -90 degrees
- moved R9 46.7 mm to (83.8, 107.7), turned to -90 degrees
- moved C8 46.1 mm to (125.7, 110.5), turned to -90 degrees
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Connections:
- C1 pad 1: Net-(FUSE1-dVdT) -> VBUSP
- C2 pad 1: VBUS_P -> VBUSP
- C4 pad 1: +3.3V -> Net-(REG2-BOOT)
- C4 pad 2: GND -> Net-(REG2-SW)
- C5 pad 1: VBUS_P -> +5V
- C6 pad 1: Net-(REG2-BOOT) -> +3.3V
- C6 pad 2: Net-(REG2-SW) -> GND
- C7 pad 1: +5V -> +3.3V
- C7 pad 2: GND -> Net-(REG2-FB)
- C8 pad 1: +5V LED -> +5V
- C8 pad 2: GND -> Net-(REG1-FB)
- C9 pad 1: VBUS -> VBUSP
- D1 pad 1: GND -> VBUS
- D1 pad 2: Net-(D1-A) -> GND
- D2 pad 1: FAULT -> VBUS
- D2 pad 2: Net-(D2-A) -> GND
- D3 pad 1: PG_3V -> VBUSP
- D4 pad 1: PG_5V -> VBUS
- D4 pad 2: Net-(D4-A) -> GND
- D5 pad 1: GND -> VBUS
- D5 pad 2: Net-(D5-A) -> GND
- D6 pad 1: VBUS -> GND
- D6 pad 2: GND -> Net-(D6-A)
- D7 pad 1: VBUS -> GND
- D7 pad 2: GND -> Net-(D7-A)
- D8 pad 1: VBUS -> GND
- D8 pad 2: GND -> Net-(D8-A)
- D9 pad 1: VBUS -> Net-(D9-K)
- L1 pad 1: +3.3V -> Net-(REG1-SW)
- L1 pad 2: Net-(REG1-SW) -> +5V
- L2 pad 1: +5V -> Net-(REG2-SW)
- L2 pad 2: Net-(REG2-SW) -> +3.3V
- POGO1 pad 1: CLK_LOW -> CLK_BUS
- POGO2 pad 1: CLK_LOW -> CLK_BUS
- POGO3 pad 5: CLK_LOW -> CLK_BUS
- POGO4 pad 5: CLK_LOW -> CLK_BUS
- R1 pad 1: VBUS -> Net-(D3-A)
- R1 pad 2: Net-(FUSE1-UVLO) -> GND
- R2 pad 1: Net-(FUSE1-UVLO) -> +5V
- R2 pad 2: Net-(FUSE1-OVP) -> Net-(REG1-FB)
- R3 pad 1: Net-(FUSE1-OVP) -> Net-(REG1-FB)
- R4 pad 1: Net-(FUSE1-ILIM) -> +3.3V
- R4 pad 2: GND -> Net-(REG2-FB)
- R5 pad 1: IMON -> Net-(REG2-FB)
- R6 pad 2: Net-(REG1-FB) -> Net-(D6-A)
- R7 pad 1: Net-(REG1-FB) -> +5V
- R7 pad 2: AGND -> Net-(D7-A)
- R8 pad 1: +5V -> CLK
- R8 pad 2: Net-(REG2-FB) -> Net-(D8-A)
- R9 pad 1: Net-(REG2-FB) -> CLK_BUS
- R9 pad 2: AGND -> Net-(D9-K)
- REG1 pad 1: PGOOD -> GND
- REG1 pad 2: Net-(REG1-FB) -> Net-(REG1-SW)
- REG1 pad 3: AGND -> VBUSP
- REG1 pad 4: PG_3V -> Net-(REG1-FB)
- REG1 pad 5: (no net) -> unconnected-(REG1-EN-Pad5)
- REG1 pad 6: Net-(REG1-SW) -> Net-(REG1-BOOT)
- REG2 pad 1: PGOOD -> GND
- REG2 pad 2: Net-(REG2-FB) -> Net-(REG2-SW)
- REG2 pad 3: AGND -> VBUSP
- REG2 pad 4: PG_5V -> Net-(REG2-FB)
- REG2 pad 5: (no net) -> unconnected-(REG2-EN-Pad5)
- REG2 pad 6: Net-(REG2-SW) -> Net-(REG2-BOOT)
Routing:
- net +3.3V: track 0.75 -> 778.1 mm, vias 13 -> 3
- net +5V: track 17.1 -> 688.7 mm, vias 2 -> 4
- net CLK_LOW: track 572.7 -> 0.00 mm, vias 2 -> 0
- net CLK_BUS: track 0.00 -> 507.9 mm, vias 0 -> 1
- net CLK: track 655.2 -> 738.5 mm, vias 2 -> 4
- net +5V LED: track 77.5 -> 0.00 mm
- net PG_3V: track 67.5 -> 0.00 mm, vias 2 -> 0
- net FAULT: track 51.0 -> 0.00 mm, vias 2 -> 0
- net PG_5V: track 46.8 -> 0.00 mm, vias 2 -> 0
- net PGOOD: track 25.7 -> 0.00 mm, vias 3 -> 0
- net GND: track 18.3 -> 23.9 mm, vias 43 -> 3
- net Net-(FUSE1-OVP): track 5.13 -> 0.00 mm
- net Net-(D9-K): track 0.00 -> 4.24 mm
- net Net-(FUSE1-UVLO): track 4.07 -> 0.00 mm
- net VBUS: track 3.96 -> 0.00 mm
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- added copper zone on F.Cu, net GND
- added copper zone on B.Cu, net VBUSP
- removed copper zone on F.Cu, net (none)
- removed copper zone on In2.Cu, net +3.3V
- removed copper zone on B.Cu, net AGND
- removed copper zone on B.Cu, net CLK
- removed copper zone on In1.Cu, net GND
- removed copper zone on B.Cu, net Net-(REG1-BOOT)
- removed copper zone on B.Cu, net Net-(REG2-BOOT)
- removed copper zone on B.Cu, net VBUS_P
Other:
- copper layers 4 -> 2
- board text added: "Minibadges: 25 In: 5V - 28V 3.25A Out: 3.3V@3A/5V@3A"
- board text removed: "Minibadges: 25 In: 5V - 28V 3.25A Out: 3.3V/5V 6A UVLO/OVP: 4.7V-32V"
- board text removed: "Pips801"

Commit message: Add test points
Parts:
- added TP1: VBUS, TestPoint:TestPoint_Pad_D1.5mm, B.Cu at (119.4, 138.6)
- added TP2: 5V, TestPoint:TestPoint_Pad_D1.5mm, B.Cu at (101.6, 138.6)
- added TP3: 3.3V, TestPoint:TestPoint_Pad_D1.5mm, B.Cu at (114.9, 138.6)
- added TP4: CLK, TestPoint:TestPoint_Pad_D1.5mm, B.Cu at (106.0, 138.6)
- added TP5: CLK_BUS, TestPoint:TestPoint_Pad_D1.5mm, B.Cu at (110.5, 138.6)
- added TP6: GND, TestPoint:TestPoint_Pad_D1.5mm, B.Cu at (110.5, 132.7)
- added kibuzzard-696F1606: G***, kibuzzard-696F1606, B.Cu at (110.5, 142.7)
Routing:
- net +3.3V: track 778.1 -> 797.7 mm
- net CLK_BUS: track 507.9 -> 526.7 mm, vias 1 -> 2
- net +5V: track 688.7 -> 700.4 mm
- net CLK: track 738.5 -> 746.5 mm
- net VBUS: track 0.00 -> 2.62 mm, vias 6 -> 7

Commit message: fix minibadge footprint
Parts:
- MB13, MB14, MB15: footprint MiniBadge:MiniBadge_Slot_Basic -> MiniBadge:MiniBadge_Slot_Reflective
