File: 5x5 Display/5x5 Display.kicad_pcb (KiCad board)
At the start: 2 copper layers, 129.5 x 129.5 mm, 87 parts, among them Q1 PMOS

Commit message: R2 Ordered
Parts:
- G***: value LOGO -> cat
- logo1: renamed from G***; value LOGO -> Beehive Logo
- moved G*** 80.1 mm to (161.5, 132.0)
- moved kibuzzard-69659941 80.1 mm to (161.5, 142.6)
- moved kibuzzard-69659724 25.4 mm to (170.2, 66.7)
- moved kibuzzard-6965973E 25.4 mm to (101.6, 66.7)
- moved logo1 25.4 mm to (118.1, 60.0)
Routing:
- net CLK: track 746.5 -> 747.8 mm
