File: 5x5 Display/minibadge_sockets.kicad_sch (KiCad schematic)
At the start: 25 parts

Commit message: Initial route complete
Parts:
- MB13, MB14, MB15: footprint MiniBadge:MiniBadge_Slot_Reflective -> MiniBadge:MiniBadge_Slot_Basic
Changed lines of the file:
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@@
 			)
 		)
-		(property "Footprint" "MiniBadge:MiniBadge_Slot_Reflective"
+		(property "Footprint" "MiniBadge:MiniBadge_Slot_Basic"
 			(at 128.27 101.6 0)
 			(effects
@@
 			)
 		)
-		(property "Footprint" "MiniBadge:MiniBadge_Slot_Reflective"
+		(property "Footprint" "MiniBadge:MiniBadge_Slot_Basic"
 			(at 162.56 101.6 0)
 			(effects
@@
 			)
 		)
-		(property "Footprint" "MiniBadge:MiniBadge_Slot_Reflective"
+		(property "Footprint" "MiniBadge:MiniBadge_Slot_Basic"
 			(at 93.98 101.6 0)
 			(effects

Commit message: R1
Parts:
- MB1, MB10, MB11, MB12, MB13, MB14, MB15, MB16, MB17, MB18, MB19, MB2, MB20, MB21, MB22, MB23, MB24, MB25, MB3, MB4, MB5, MB6, MB7, MB8, MB9: now left out of the parts list
Changed lines of the file:
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@@
 		(unit 1)
 		(exclude_from_sim no)
-		(in_bom yes)
+		(in_bom no)
 		(on_board yes)
 		(dnp no)
@@
 		(unit 1)
 		(exclude_from_sim no)
-		(in_bom yes)
+		(in_bom no)
 		(on_board yes)
 		(dnp no)
@@
 		(unit 1)
 		(exclude_from_sim no)
-		(in_bom yes)
+		(in_bom no)
 		(on_board yes)
 		(dnp no)
@@
 		(unit 1)
 		(exclude_from_sim no)
-		(in_bom yes)
+		(in_bom no)
 		(on_board yes)
 		(dnp no)
@@
 		(unit 1)
 		(exclude_from_sim no)
-		(in_bom yes)
+		(in_bom no)
 		(on_board yes)
 		(dnp no)
@@
 		(unit 1)
 		(exclude_from_sim no)
-		(in_bom yes)
+		(in_bom no)
 		(on_board yes)
 		(dnp no)
@@
 		(unit 1)
 		(exclude_from_sim no)
-		(in_bom yes)
+		(in_bom no)
 		(on_board yes)
 		(dnp no)
@@
 		(unit 1)
 		(exclude_from_sim no)
-		(in_bom yes)
+		(in_bom no)
 		(on_board yes)
 		(dnp no)
@@
 		(unit 1)
 		(exclude_from_sim no)
-		(in_bom yes)
+		(in_bom no)
 		(on_board yes)
 		(dnp no)
@@
 		(unit 1)
 		(exclude_from_sim no)
-		(in_bom yes)
+		(in_bom no)
 		(on_board yes)
 		(dnp no)
@@
 		(unit 1)
 		(exclude_from_sim no)
-		(in_bom yes)
+		(in_bom no)
 		(on_board yes)
 		(dnp no)
@@
 		(unit 1)
 		(exclude_from_sim no)
-		(in_bom yes)
+		(in_bom no)
 		(on_board yes)
 		(dnp no)
@@
 		(unit 1)
 		(exclude_from_sim no)
-		(in_bom yes)
+		(in_bom no)
 		(on_board yes)
 		(dnp no)
@@
 		(unit 1)
 		(exclude_from_sim no)
-		(in_bom yes)
+		(in_bom no)
 		(on_board yes)
 		(dnp no)
@@
 		(unit 1)
 		(exclude_from_sim no)
-		(in_bom yes)
+		(in_bom no)
 		(on_board yes)
 		(dnp no)
@@
 		(unit 1)
 		(exclude_from_sim no)
-		(in_bom yes)
+		(in_bom no)
 		(on_board yes)
 		(dnp no)
@@
 		(unit 1)
 		(exclude_from_sim no)
-		(in_bom yes)
+		(in_bom no)
 		(on_board yes)
 		(dnp no)
@@
 		(unit 1)
 		(exclude_from_sim no)
-		(in_bom yes)
+		(in_bom no)
 		(on_board yes)
 		(dnp no)
@@
 		(unit 1)
 		(exclude_from_sim no)
-		(in_bom yes)
+		(in_bom no)
 		(on_board yes)
 		(dnp no)
@@
 		(unit 1)
 		(exclude_from_sim no)
-		(in_bom yes)
+		(in_bom no)
 		(on_board yes)
 		(dnp no)
@@
 		(unit 1)
 		(exclude_from_sim no)
-		(in_bom yes)
+		(in_bom no)
 		(on_board yes)
 		(dnp no)
@@
 		(unit 1)
 		(exclude_from_sim no)
-		(in_bom yes)
+		(in_bom no)
 		(on_board yes)
 		(dnp no)
@@
 		(unit 1)
 		(exclude_from_sim no)
-		(in_bom yes)
+		(in_bom no)
 		(on_board yes)
 		(dnp no)
@@
 		(unit 1)
 		(exclude_from_sim no)
-		(in_bom yes)
+		(in_bom no)
 		(on_board yes)
 		(dnp no)
@@
 		(unit 1)
 		(exclude_from_sim no)
-		(in_bom yes)
+		(in_bom no)
 		(on_board yes)
 		(dnp no)

Commit message: fix minibadge footprint
Parts:
- MB13, MB14, MB15: footprint MiniBadge:MiniBadge_Slot_Basic -> MiniBadge:MiniBadge_Slot_Reflective
Changed lines of the file:
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@@
 			)
 		)
-		(property "Footprint" "MiniBadge:MiniBadge_Slot_Basic"
+		(property "Footprint" "MiniBadge:MiniBadge_Slot_Reflective"
 			(at 128.27 101.6 0)
 			(effects
@@
 			)
 		)
-		(property "Footprint" "MiniBadge:MiniBadge_Slot_Basic"
+		(property "Footprint" "MiniBadge:MiniBadge_Slot_Reflective"
 			(at 162.56 101.6 0)
 			(effects
@@
 			)
 		)
-		(property "Footprint" "MiniBadge:MiniBadge_Slot_Basic"
+		(property "Footprint" "MiniBadge:MiniBadge_Slot_Reflective"
 			(at 93.98 101.6 0)
 			(effects
