File: Minibadge PD module/Minibadge PD module.kicad_sch (KiCad schematic)
At the start: 16 parts, among them J1 USB_C_Receptacle_USB2.0_14P, J2 Conn_01x05, U1 TPD4E05U06DQA, U2 HUSB238A-xxxxx-QN16R, U3 TPS54331, U4 74HC4060

Commit message: PD module work
Parts:
- removed D1: D1, symbol Device:D_Schottky_Small
- removed U3: TPS54331, Package_SO:TI_SO-PowerPAD-8_ThermalVias, symbol Regulator_Switching:TPS54336ADDA
- added C10, C9: 10μF 50V, Capacitor_SMD:C_1206_3216Metric, symbol Device:C_Small
- added C6: *10nF, Capacitor_SMD:C_0603_1608Metric, symbol Device:C_Small
- added C7, C8: 100nF, Capacitor_SMD:C_0603_1608Metric, symbol Device:C_Small
- added D1, D8: ≥28V TVS, Diode_SMD:D_SMA, symbol Device:D_TVS_Small
- added D4: VBUS, LED_SMD:LED_0603_1608Metric, symbol Device:LED_Small
- added D5: CLK, LED_SMD:LED_0603_1608Metric, symbol Device:LED_Small
- added D6: PD FAULT, LED_SMD:LED_0603_1608Metric, symbol Device:LED_Small
- added D7: FUSE FAULT, LED_SMD:LED_0603_1608Metric, symbol Device:LED_Small
- added R10, R11, R12, R13, R14, R15, R16: *, Resistor_SMD:R_0603_1608Metric, symbol Device:R_Small
- added R2: 900kΩ, Resistor_SMD:R_0603_1608Metric, symbol Device:R_Small
- added R5: 24kΩ, Resistor_SMD:R_0603_1608Metric, symbol Device:R_Small
- added R6: *11kΩ, Resistor_SMD:R_0603_1608Metric, symbol Device:R_Small
- added R7: 8.45kΩ, Resistor_SMD:R_0603_1608Metric, symbol Device:R_Small
- added R8: 20kΩ, Resistor_SMD:R_0603_1608Metric, symbol Device:R_Small
- added R9: 10kΩ, Resistor_SMD:R_0603_1608Metric, symbol Device:R_Small
- added SW1: Fast/Slow, symbol Switch:SW_SPDT
- added SW2: Reset, symbol Switch:SW_Push
- added U3: ETA2845S2G, Package_TO_SOT_SMD:TSOT-23-6, symbol Regulator_Switching:LM2841X
- added U4: MX26631DL, Package_DFN_QFN:QFN-24-1EP_4x4mm_P0.5mm_EP2.6x2.6mm_ThermalVias, symbol MX26631DL:MX26631DL
- added U5: DRV8837C, Package_SON:WSON-8-1EP_2x2mm_P0.5mm_EP0.9x1.6mm, symbol Driver_Motor:DRV8837C
- C1: value C1 -> 10μF 50V; footprint (none) -> Capacitor_SMD:C_1206_3216Metric
- C2: value C2 -> 100nF; footprint (none) -> Capacitor_SMD:C_0603_1608Metric
- C3: value Cboot -> 1μF 50V; footprint (none) -> Capacitor_SMD:C_0603_1608Metric
- C4: value Css -> 100pF; footprint (none) -> Capacitor_SMD:C_0603_1608Metric
- C5: value Cboot -> 22uF; footprint (none) -> Capacitor_SMD:C_1206_3216Metric
- J1: value USB_C_Receptacle_USB2.0_14P -> USB-C port; footprint (none) -> Connector_USB:USB_C_Receptacle_HRO_TYPE-C-31-M-12
- J2: footprint (none) -> Connector_PinHeader_2.54mm:PinHeader_1x05_P2.54mm_Horizontal
- L1: value Lo -> 10μH; footprint (none) -> Inductor_SMD:L_Taiyo-Yuden_MD-3030; LCSC Part # (none) -> C668449
- R1: value R3 -> 75kΩ; footprint (none) -> Resistor_SMD:R_0603_1608Metric
- R3: value Ro1 -> Rvset; footprint (none) -> Resistor_SMD:R_0603_1608Metric; now not fitted
- R4: value Ro2 -> Riset; footprint (none) -> Resistor_SMD:R_0603_1608Metric; now not fitted
- U2: value HUSB238A-xxxxx-QN16R -> HUSB238A
- U6: renamed from U4; footprint (none) -> Package_SO:TSSOP-16_4.4x5mm_P0.65mm
Connections:
- net +3.3V: now also C4.2, C5.2, R1.1, U2.5 (VDD), U6.16 (VDD), C8.1, R11.2, R14.2, U5.1 (VM), U5.6 (IN1), U5.7 (~{SLEEP}), U5.8 (VCC); no longer C5.1, R3.1
- net CC1: now also U1.4 (D2+), U1.7 (NC)
- net CC2: now also U1.5 (D2-), U1.6 (NC)
- net D+: now also U1.1 (D1+), U1.10 (NC)
- net D-: now also U1.2 (D1-), U1.9 (NC)
- net GND: now also C1.2, C3.1, C5.1, J1.A1 (GND), J1.A12 (GND), J1.B1 (GND), J1.B12 (GND), J1.S1 (SHIELD), J2.3 (Pin_3), J2.4 (Pin_4), R3.2, R4.1, U1.3 (GND), U1.8 (GND), U2.12 (~{EN}), U2.17 (GND), U6.12 (CLR), U6.8 (VSS), C10.2, C6.2, C8.2, C9.2, D1.2 (A2), D4.1 (K), D5.1 (K), D6.1 (K), D8.2 (A2), R16.2, R2.1, R5.2, R6.2, R9.2, SW2.2, U3.2 (GND), U4.11 (MODE), U4.25 (PowerPAD), U4.8 (GND), U5.4 (GND), U5.9 (GND); no longer C2.2, C4.2, C5.2, R1.2, R4.2
- net VBUS: now also C1.1, C3.2, C10.1, D1.1 (A1), R10.1, U3.4 (EN), U3.5 (VIN), U4.1 (IN), U4.2 (IN), U4.5 (IN_SYS)
- net at L1.1: now also C2.2, U3.6 (SW); no longer C3.2
- net at C2.1: now also U3.1 (BOOST); no longer C1.1
- net at C4.1: now also R1.2, R5.1, U3.3 (FB)
- net at U6.10 (Φ0): now also R7.2
- net at U6.11 (~{Φ1}): now also R8.2
- net SLOW: now reaches U6.13 (Q9)
- net SLOW: now also SW1.3 (C)
- net FAST: now reaches U6.14 (Q8)
- net FAST: now also SW1.1 (A)
- net at U6.9 (~{Φ0}): now also C7.2
- net at U2.10 (SCL/SNK_ISET): now also R4.2
- net PD_FAULT: now reaches U2.13 (FAULT/OUT2)
- net PD_FAULT: now also R13.2
- net at U2.6 (~{DEBUG}): now also R2.2
- net at U2.9 (SDA/SNK_VSET): now also R3.1
- net VBUSP: now reaches J2.1 (Pin_1)
- net VBUSP: now also J2.2 (Pin_2), C9.1, D8.1 (A1), U4.17 (OUT), U4.18 (OUT)
- net CLK_BUS: now reaches J2.5 (Pin_5)
- net CLK_BUS: now also U5.2 (OUT1)
- new net: R10.2, R15.1, U4.6 (UVLO)
- new net: R6.1, U4.10 (ILIM)
- new net: R15.2, R16.1, U4.7 (OVP)
- new net: C6.1, U4.9 (dVdT)
- new net: D7.2 (A), R14.1
- new net: D4.2 (A), R11.1
- new net: D5.2 (A), R12.1
- new net: D6.2 (A), R13.1
- new net: C7.1, R7.1, R8.1
- new net CLK_LOW: R12.2, SW1.2 (B), U5.5 (IN2)
- new net FUSE_FAULT: D7.1 (K), U4.14 (FLT)
- new net IMON: R9.1, U4.13 (IMON)
- new net SHUTDOWN: SW2.1, U4.12 (SHDN)
- no-connect marks 1 -> 18
Other:
- note added: "3.3V 400mA output"
- note added: "Configured for 28V 3.25A PDO"
- note added: "Notes * Protect CLK_BUS * Determine FET for VBUS gate (or remove) * Wire RESET button * Wire e-fuse * Wire clock speed switch"
- note added: "OVP UVLO ILIM"
- company: (none) -> Beehive Engineering
- title: (none) -> Minibadge Display PD Module
- moved on the sheet: J1, J2, U1, U2, U6
